File: pcb.kicad_pcb (KiCad board)
At the start: 4 copper layers, 8.6 x 5 mm, 80 parts, among them IC1 XCL103D503CR-G, IC10 ADG801BRTZ-REEL7, IC2 MCP659-E_ML, IC3 DS4424N+T&R, IC4 W25Q16JVUXIQ, IC5 TC42X-2-102E, IC6 TC42X-2-102E, IC7 TC42X-2-102E, IC8 TC42X-2-102E, IC9 AD8403ARUZ1-REEL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

Commit message: WIP
Parts:
- J1: footprint 2171790001:2171790001_MOL -> my_2171790001:2171790001
- J2, J3: footprint Connector_PinHeader_1.27mm:PinHeader_1x04_P1.27mm_Vertical -> conn:PinHeader_1x04_P1.27mm_Vertical
- J4: footprint Connector_PinHeader_1.27mm:PinHeader_1x02_P1.27mm_Vertical -> conn:PinHeader_1x02_P1.27mm_Vertical
- J5: footprint Connector_PinHeader_1.27mm:PinHeader_1x03_P1.27mm_Vertical -> conn:PinHeader_1x03_P1.27mm_Vertical
- moved J1 4.78 mm to (43.6, 42.4)
Other:
- board outline removed

Commit message: WIP
Parts:
- C13, C14, C15, C16, C17, C2, C20, C21, C22, C23, C24, C25, C4, C8, C9, R19, R20, R7, R8: moved to B.Cu
- moved R1 159.7 mm to (191.9, 85.9), turned to 90 degrees
- moved J1 156.7 mm to (195.3, 81.5), turned to 90 degrees
- moved J2 151.3 mm to (190.2, 78.4)
- moved R2 149.8 mm to (193.6, 76.9), turned to 90 degrees
- moved R18 109.2 mm to (178.8, 102.7)
- moved C12 109.2 mm to (185.7, 105.7)
- moved LED1 109.2 mm to (183.1, 105.7)
- moved R13 109.2 mm to (176.3, 109.7)
- moved Q1 96.1 mm to (130.4, 41.6)
- moved Q2 96.1 mm to (125.9, 55.8)
- moved Q3 96.1 mm to (134.0, 71.6)
- moved Q4 96.1 mm to (127.3, 88.9)
- moved R24 96.1 mm to (132.6, 41.3)
- moved R26 96.1 mm to (127.8, 70.2)
- moved R28 96.1 mm to (127.8, 73.7)
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Other:
- board outline added: 30 x 22 mm

Commit message: WIP
Parts:
- C10, C11, C18, C19, C5, C6, C7, R10, R11, R12, R14, R15, R16, R17, R21, R3, R4, R5, R6, R9: moved to B.Cu
- moved D1 43.4 mm to (175.7, 85.0)
- moved R6 38.1 mm to (158.0, 105.8), turned to -90 degrees
- moved C18 37.5 mm to (185.5, 25.1), turned to -90 degrees
- moved R5 37.3 mm to (157.3, 105.8), turned to -90 degrees
- moved R21 32.3 mm to (187.0, 33.6), turned to 180 degrees
- moved IC10 31.9 mm to (186.5, 26.0), turned to 90 degrees
- moved R4 31.5 mm to (156.6, 105.8), turned to -90 degrees
- moved C19 31.2 mm to (186.7, 34.6), turned to 90 degrees
- moved R3 30.7 mm to (155.9, 105.8), turned to 90 degrees
- moved R17 27.0 mm to (147.5, 101.2), turned to 180 degrees
- moved IC3 26.8 mm to (156.4, 103.9), turned to 90 degrees
- moved R10 26.5 mm to (157.1, 101.2), turned to 180 degrees
- moved R15 23.9 mm to (153.9, 101.2), turned to 180 degrees
- moved C11 23.0 mm to (147.5, 100.5), turned to 180 degrees
- moved C6 22.7 mm to (157.1, 100.5), turned to 180 degrees
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Connections:
- C6 pad 1: /VOUTA -> /SPX_RAW
- C6 pad 2: /SPX_RAW -> /VOUTA
- J3 pad 1: /USB_VBUS_ -> /USB_DP_
- J3 pad 2: GND -> /USB_DN_
- J3 pad 3: /USB_DP_ -> GND
- J3 pad 4: /USB_DN_ -> /USB_VBUS_
Routing:
- net /C4_RAW: track 0.00 -> 16.3 mm, vias 0 -> 1
- net GND: track 0.00 -> 11.5 mm, vias 0 -> 7
- net /VIN: track 0.00 -> 11.0 mm
- net +3V3: track 0.00 -> 10.8 mm, vias 0 -> 12
- net /VOUTD: track 0.00 -> 10.5 mm, vias 0 -> 2
- net /VOUTA: track 0.00 -> 10.4 mm, vias 0 -> 2
- net /C2_RAW: track 0.00 -> 9.40 mm, vias 0 -> 2
- net /3DS_C4: track 0.00 -> 9.29 mm, vias 0 -> 1
- net /3DS_SPX: track 0.00 -> 8.24 mm, vias 0 -> 1
- net /SPX_RAW: track 0.00 -> 8.21 mm, vias 0 -> 2
- net /3DS_SPY: track 0.00 -> 6.93 mm, vias 0 -> 1
- net /3DS_C2: track 0.00 -> 6.87 mm, vias 0 -> 1
- net /SPY_RAW: track 0.00 -> 6.25 mm, vias 0 -> 2
- net +5V: track 0.00 -> 5.63 mm, vias 0 -> 2
- net /QSPI_SS: track 0.00 -> 4.72 mm, vias 0 -> 1
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
Commit message: WIP
Parts:
- moved IC10 62.6 mm to (153.2, 78.9)
- moved C18 62.6 mm to (152.2, 78.0)
- moved IC9 62.6 mm to (155.6, 85.0)
- moved C19 62.6 mm to (153.4, 87.6)
- moved R21 62.6 mm to (153.7, 86.5)
- moved C11 26.9 mm to (153.9, 74.4)
- moved R17 26.9 mm to (153.9, 75.1)
- moved C7 26.9 mm to (157.1, 74.4)
- moved R12 26.9 mm to (157.1, 75.1)
- moved C10 26.9 mm to (160.3, 74.4)
- moved R15 26.9 mm to (160.3, 75.1)
- moved C6 26.9 mm to (163.5, 74.4)
- moved R10 26.9 mm to (163.5, 75.1)
- moved C5 26.7 mm to (161.7, 76.1)
- moved IC3 26.7 mm to (162.5, 77.9)
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Connections:
- R16 pad 1: Net-(IC8-WIPER) -> /3DS_C4
- R16 pad 2: /3DS_C4 -> Net-(IC8-WIPER)
Routing:
- net /AGND: track 0.00 -> 12.6 mm, vias 0 -> 5
- net Net-(IC9-B4): track 0.00 -> 7.59 mm
- net /C2_RAW: track 9.40 -> 16.7 mm
- net Net-(IC9-A4): track 0.00 -> 5.92 mm
- net Net-(IC10-S): track 0.00 -> 5.04 mm, vias 0 -> 2
- net Net-(IC10-D): track 0.00 -> 3.27 mm, vias 0 -> 2
- net /SPY_RAW: track 6.25 -> 9.34 mm
- net /XIN: track 0.00 -> 3.00 mm
- net /VOUTC: track 4.33 -> 2.08 mm, vias 2 -> 1
- net /C4_RAW: track 16.3 -> 14.1 mm, vias 1 -> 2
- net /VOUTA: track 10.4 -> 8.46 mm
- net /VOUTD: track 10.5 -> 8.81 mm
- net /3DS_SPY: track 6.93 -> 5.69 mm
- net /XOUT: track 0.00 -> 1.23 mm, vias 0 -> 1
- net Net-(Y1-OUTPUT): track 0.00 -> 1.22 mm, vias 0 -> 1
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
Commit message: WIP
Parts:
- C12, R13, R18, R22, R23, R24, R25, R26, R27, R28, R29: moved to B.Cu
- moved R22 58.9 mm to (164.0, 87.6), turned to 0 degrees
- moved Q1 57.7 mm to (163.9, 88.6), turned to 180 degrees
- moved R24 55.7 mm to (162.1, 88.6), turned to 0 degrees
- moved R23 52.0 mm to (164.0, 84.2)
- moved R25 49.0 mm to (162.1, 85.2)
- moved Q2 48.0 mm to (163.9, 85.2), turned to 180 degrees
- moved R27 47.4 mm to (168.7, 85.4), turned to 90 degrees
- moved R29 46.6 mm to (167.6, 86.0), turned to 180 degrees
- moved Q4 40.6 mm to (167.7, 86.0), turned to 180 degrees
- moved R26 37.7 mm to (164.0, 80.8)
- moved R28 35.2 mm to (162.1, 81.8)
- moved D2 31.8 mm to (183.7, 78.6), turned to 90 degrees
- moved Q3 31.6 mm to (163.9, 81.8), turned to 180 degrees
- moved C12 29.7 mm to (167.6, 82.2), turned to 90 degrees
- moved LED1 27.7 mm to (167.1, 83.0), turned to 90 degrees
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Routing:
- net +5V: track 6.28 -> 26.2 mm, vias 3 -> 8
- net +3.3V: track 0.41 -> 11.4 mm, vias 1 -> 9
- net /SPI_CS_5V: track 0.00 -> 10.2 mm, vias 0 -> 3
- net /SPI_TX_5V: track 0.00 -> 9.94 mm, vias 0 -> 1
- net /SPI_SCK_5V: track 0.00 -> 9.31 mm, vias 0 -> 1
- net /VIN: track 11.0 -> 5.44 mm
- net Net-(U2-USB_DM): track 0.89 -> 2.35 mm
- net Net-(U2-USB_DP): track 0.88 -> 1.66 mm
- net GND: track 12.2 -> 12.9 mm, vias 17 -> 18
- net Net-(IC10-D): track 3.27 -> 3.94 mm
- net Net-(IC10-S): track 5.04 -> 5.71 mm
- net Net-(LED1-DOUT): track 0.00 -> 0.26 mm, vias 0 -> 1
- net Net-(LED1-DIN): track 0.00 -> 0.22 mm, vias 0 -> 1
- net /SPI_TX: vias 0 -> 1
- net /SPI_SCK: vias 0 -> 1
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
Commit message: WIP
Parts:
- C4, C8: moved to F.Cu
- Q1, Q2, Q3: moved to B.Cu
- moved D2 10.7 mm to (177.6, 87.4)
- moved J1 10.7 mm to (184.7, 83.1)
- moved R2 9.71 mm to (184.2, 79.3)
- moved R26 9.70 mm to (155.7, 85.8)
- moved R28 9.13 mm to (153.3, 84.1), turned to 90 degrees
- moved Q3 8.53 mm to (155.6, 83.7)
- moved R1 7.77 mm to (184.2, 86.8), turned to -90 degrees
- moved J2 7.72 mm to (183.0, 81.2)
- moved R29 5.62 mm to (164.7, 81.2), turned to -90 degrees
- moved R27 5.32 mm to (165.4, 81.2)
- moved Q1 4.91 mm to (164.7, 83.7)
- moved R13 4.72 mm to (163.4, 85.8), turned to 180 degrees
- moved R24 4.54 mm to (162.4, 84.1), turned to 90 degrees
- moved R25 4.43 mm to (157.9, 84.1), turned to 90 degrees
- moved C4 4.25 mm to (168.4, 86.3)
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Connections:
- C4 pad 1: +3.3V -> +3V3
- J2 pad 1: /USB_VBUS -> /USB_DP
- J2 pad 2: /USB_GND -> /USB_DN
- J2 pad 3: /USB_DP -> /USB_GND
- J2 pad 4: /USB_DN -> /USB_VBUS
- J6 pad 1: /3DS_BTN0 -> GND
- J6 pad 10: /3DS_BTN9 -> /3DS_TSXM
- J6 pad 11: /3DS_BTN10 -> /3DS_TSXP
- J6 pad 12: /3DS_BTN11 -> /3DS_C4
- J6 pad 13: /3DS_BTN12 -> /3DS_C2
- J6 pad 14: /3DS_BTN13 -> /3DS_SPY
- J6 pad 15: /3DS_BTN14 -> /3DS_SPX
- J6 pad 16: /3DS_BTN15 -> /3DS_BTN14
- J6 pad 17: /3DS_SPX -> /3DS_BTN12
- J6 pad 18: /3DS_SPY -> /3DS_BTN13
- J6 pad 19: /3DS_C2 -> /3DS_BTN11
- J6 pad 2: /3DS_BTN1 -> GND
- J6 pad 20: /3DS_C4 -> /3DS_BTN10
- J6 pad 21: /3DS_TSXP -> /3DS_BTN9
- J6 pad 22: /3DS_TSXM -> /3DS_BTN8
- J6 pad 23: /3DS_TSYP -> /3DS_BTN7
- J6 pad 24: /3DS_TSYM -> /3DS_BTN6
- J6 pad 25: /3DS_VBUS -> /3DS_BTN5
- J6 pad 26: /3DS_VBUS -> /3DS_BTN4
- J6 pad 27: /3DS_VBUS -> /3DS_BTN3
- J6 pad 28: GND -> /3DS_BTN2
- J6 pad 29: GND -> /3DS_BTN1
- J6 pad 3: /3DS_BTN2 -> GND
- J6 pad 30: GND -> /3DS_BTN0
- J6 pad 4: /3DS_BTN3 -> /3DS_VBUS
- J6 pad 5: /3DS_BTN4 -> /3DS_VBUS
- J6 pad 6: /3DS_BTN5 -> /3DS_VBUS
- J6 pad 7: /3DS_BTN6 -> /3DS_BTN15
- J6 pad 8: /3DS_BTN7 -> /3DS_TSYM
- J6 pad 9: /3DS_BTN8 -> /3DS_TSYP
- Q1 pad 1: +3.3V -> +3V3
- Q2 pad 1: +3.3V -> +3V3
- Q3 pad 1: +3.3V -> +3V3
- Q4 pad 1: +3.3V -> +3V3
- R22 pad 1: +3.3V -> +3V3
- R23 pad 1: +3.3V -> +3V3
- R26 pad 1: +3.3V -> +3V3
- R27 pad 1: +3.3V -> +3V3
- U1 pad 1: +3.3V -> +3V3
- U2 pad 27: /I2C_SDA -> /I2C_SCL
- U2 pad 28: /I2C_SCL -> /I2C_SDA
- U2 pad 29: /SPI_SCK -> /LED_DIN
- U2 pad 30: /SPI_TX -> /SPST_IN
- U2 pad 31: /SPI_CS -> /SPI_SCK
- U2 pad 32: /SPST_IN -> /SPI_TX
- U2 pad 34: /LED_DIN -> /SPI_CS
Routing:
- net +3V3: track 10.8 -> 85.9 mm, vias 12 -> 15
- net /SPI_TX: track 0.00 -> 24.8 mm, vias 1 -> 4
- net +5V: track 26.2 -> 46.7 mm, vias 8 -> 7
- net /SPST_IN: track 0.00 -> 18.2 mm, vias 1 -> 2
- net /3DS_VBUS: track 0.00 -> 16.5 mm, vias 0 -> 3
- net /3DS_C4: track 8.27 -> 24.1 mm, vias 1 -> 2
- net /SPI_CS: track 0.00 -> 14.6 mm, vias 1 -> 2
- net /3DS_C2: track 7.01 -> 18.8 mm, vias 1 -> 2
- net +3.3V: track 11.4 -> 0.00 mm, vias 9 -> 0
- net /SPI_SCK: track 0.00 -> 9.98 mm, vias 1 -> 2
- net /USB_VBUS: track 0.00 -> 9.75 mm
- net /SWCLK: track 0.00 -> 9.46 mm, vias 0 -> 1
- net GND: track 12.9 -> 21.6 mm, vias 18 -> 30
- net /I2C_SDA: track 0.00 -> 8.50 mm
- net /3DS_SPY: track 5.69 -> 14.0 mm
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- added copper zone on B.Cu, net /USB_GND
- added copper zone on F.Cu, net /USB_GND
- added copper zone on B.Cu, net GND
- added copper zone on F.Cu, net GND
- added copper zone on In1.Cu, net GND
Other:
- board size 30 x 22 mm -> 39.2 x 17.9 mm

Commit message: WIP
Parts:
- added REF**: MouseBites_2.54, MouseBites_2.54:MouseBites_2.54, F.Cu at (180.3, 83.1)
- moved C9 2.22 mm to (176.5, 78.5), turned to 180 degrees
- moved J2 1.40 mm to (184.4, 81.2)
- moved R1 1.40 mm to (185.6, 86.8)
- moved R2 1.40 mm to (185.6, 79.3)
- moved J1 1.39 mm to (186.1, 83.1)
Connections:
- J6 pad 10: /3DS_TSXM -> /3DS_TSYP
- J6 pad 11: /3DS_TSXP -> /3DS_TSYM
- J6 pad 8: /3DS_TSYM -> /3DS_TSXP
- J6 pad 9: /3DS_TSYP -> /3DS_TSXM
Routing:
- net /3DS_TSXM: track 0.00 -> 23.5 mm, vias 1 -> 3
- net /3DS_TSXP: track 0.00 -> 22.9 mm, vias 0 -> 3
- net /3DS_TSYM: track 0.00 -> 15.2 mm, vias 0 -> 2
- net /3DS_TSYP: track 0.00 -> 15.1 mm, vias 0 -> 2
- net /3DS_VBUS: track 16.5 -> 19.4 mm
- net /USB_GND: track 6.86 -> 5.25 mm
- net /AGND: track 14.1 -> 15.4 mm
- net +3V3: track 85.9 -> 86.8 mm
- net /VOUTA: track 8.46 -> 7.93 mm
- net GND: track 21.6 -> 21.7 mm, vias 30 -> 29
- added copper zone on In2.Cu, net +1V1
- added copper zone on In2.Cu, net +3V3
- added copper zone on In2.Cu, net +5V
- added copper zone on In2.Cu, net /3DS_VBUS
- added copper zone on In1.Cu, net /AGND
- added copper zone on F.Cu, net /VIN
Other:
- board size 39.2 x 17.9 mm -> 40.6 x 17.9 mm
