File: pcb.kicad_sch (KiCad schematic)
At the start: 9 parts, among them IC1 XCL103D503CR-G, J1 2171790001, U1 NCP167AMX330TBG

Commit message: WIP
Parts:
- added C1, C12, C13, C2, C21, C22: 100n, Capacitor_SMD:C_0402_1005Metric, symbol Device:C_Small
- added C10, C11, C4, C5, C6, C7, C8, C9: 1u, symbol Device:C_Small
- added C18, C19, C23, C24: 10n, Capacitor_SMD:C_0603_1608Metric, symbol Device:C_Small
- added C20, C25: 100n, Capacitor_SMD:C_0603_1608Metric, symbol Device:C_Small
- added C3: 1u, Capacitor_SMD:C_0402_1005Metric, symbol Device:C_Small
- added IC1: W25Q16JVUXIQ, SON50P300X200X60-9N, symbol W25Q16JVUXIQ:W25Q16JVUXIQ
- added IC10: DS4424N+T&R, DS4424N+T&R:SON40P300X300X80-15N, symbol DS4424N+T&R:DS4424N+T&R
- added IC3, IC4, IC7, IC8: TC42X-2-102E, TC42X2102E, symbol TC42X-2-102E:TC42X-2-102E
- added IC5: AD8403ARUZ1-REEL, SOP65P640X120-24N, symbol AD8403ARUZ1-REEL:AD8403ARUZ1-REEL
- added IC6: MCP659-E_ML, QFN65P400X400X100-17N-D, symbol MCP659-E_ML:MCP659-E_ML
- added IC9: ADG801BRTZ-REEL7, SOT95P280X145-6N, symbol ADG801BRTZ-REEL7:ADG801BRTZ-REEL7
- added J1: Conn_01x02, symbol Connector_Generic:Conn_01x02
- added J3, J4: Conn_01x04, symbol Connector_Generic:Conn_01x04
- added J5: Conn_01x03, symbol Connector_Generic:Conn_01x03
- added LED1: SK6805-EC15, SK6805EC15, symbol SK6805-EC15:SK6805-EC15
- added Q1, Q2, Q3, Q4: BSS138, Package_TO_SOT_SMD:SOT-23, symbol Transistor_FET:BSS138
- added R1, R3: 5.1k, symbol Device:R_Small
- added R10, R11, R12, R16, R17, R18, R19, R9: 10k, symbol Device:R_Small
- added R13: 0, symbol Device:R_Small
- added R14, R15: 1.2k, symbol Device:R_Small
- added R2: 1k, Resistor_SMD:R_0402_1005Metric, symbol Device:R_Small
- added R20, R21, R7, R8: 750, Resistor_SMD:R_0603_1608Metric, symbol Device:R_Small
- added R22, R23: 43, symbol Device:R_Small
- added R24, R25: 160k, Resistor_SMD:R_0603_1608Metric, symbol Device:R_Small
- added R26, R27: 43k, Resistor_SMD:R_0603_1608Metric, symbol Device:R_Small
- added R4, R5: 27, Resistor_SMD:R_0402_1005Metric, symbol Device:R
- added R6: 1k, symbol Device:R_Small
- added U1: RP2040, Package_DFN_QFN:QFN-56-1EP_7x7mm_P0.4mm_EP3.2x3.2mm, symbol MCU_RaspberryPi:RP2040
- added Y1: AWSCR-12.00CELA-C10-T3, AWSCR1200CELAC33T3, symbol AWSCR-12_00CELA-C33-T3:AWSCR-12.00CELA-C33-T3
- renumbered C3 to C14, C4 to C15, C1 to C16, C2 to C17, IC1 to IC2, J1 to J2, U1 to U2
Connections:
- net +3.3V: now also Q1.1 (G), Q2.1 (G), Q3.1 (G), Q4.1 (G), R11.1, R16.1, R18.1, R9.1
- net +5V: now also C13.1, C21.1, IC5.10 (~{SHDN}), IC5.15 (~{RS}), IC5.16 (VDD), LED1.2 (VDD), R10.1, R12.1, R17.1, R19.1
- net GND: now also C1.2, C10.2, C11.2, C12.2, C13.2, C2.2, C20.1, C21.2, C22.2, C25.2, C3.2, C4.2, C5.2, C6.2, C7.2, C8.2, C9.2, IC1.4 (GND), IC1.9 (EP), IC10.11 (A1), IC10.15 (EP), IC10.3 (GND), IC10.9 (A0), IC5.9 (DGND), IC6.11 (VSS), IC6.17 (EP), IC9.3 (GND), J1.1 (Pin_1), J4.2 (Pin_2), J5.2 (Pin_2), LED1.4 (GND), R13.2, R24.2, R25.1, R26.1, R27.1, U1.19 (TESTEN), U1.57 (GND), Y1.2 (GROUND)
- net 3DS_VBUS: now reaches D2.2 (A)
- net USB_GND: now reaches J2.A1/B12 (GND)
- net USB_GND: now also J2.B1/A12 (GND), J3.2 (Pin_2), R1.2, R3.2
- net USB_VBUS: now reaches J2.A4/B9 (VBUS)
- net USB_VBUS: now also J2.B4/A9 (VBUS), J3.1 (Pin_1)
- net at J2.A5 (CC1): now also R1.1
- net USB_DP: now reaches J2.A6 (DP1)
- net USB_DP: now also J2.B6 (DP2), J3.3 (Pin_3)
- net USB_DN: now reaches J2.A7 (DN1)
- net USB_DN: now also J2.B7 (DN2), J3.4 (Pin_4)
- net at J2.B5 (CC2): now also R3.1
- net USB_VBUS_: now reaches D1.2 (A)
- net USB_VBUS_: now also J4.1 (Pin_1)
- new net: IC10.5 (FS2(N.C.)), R25.2
- new net: IC5.8 (W4), IC9.1 (D)
- new net: IC5.4 (W2), IC9.2 (S)
- new net: IC8.2 (WIPER), R21.1
- new net: IC7.2 (WIPER), R20.2
- new net: IC3.2 (WIPER), R7.2
- new net: R5.2, U1.46 (USB_DM)
- new net: R4.2, U1.47 (USB_DP)
- new net: R6.2, Y1.3 (OUTPUT)
- new net: J1.2 (Pin_2), R2.1
- new net: IC10.4 (FS3(N.C.)), R24.1
- new net: IC5.18 (W3), IC5.7 (A4)
- new net: IC5.22 (W1), IC5.6 (B4)
- new net: IC4.2 (WIPER), R8.2
- new net: IC10.6 (FS1), R26.2
- new net: IC10.7 (FS0), R27.2
- new net +1V1: C1.1, C2.1, C3.1, U1.23 (DVDD), U1.45 (VREG_VOUT), U1.50 (DVDD)
- new net +3V3: C10.1, C11.1, C12.1, C20.2, C22.1, C25.1, C4.1, C5.1, C6.1, C7.1, C8.1, C9.1, IC1.8 (VCC), IC10.13 (VCC), IC6.3 (VDD), IC9.6 (VDD), U1.1 (IOVDD), U1.10 (IOVDD), U1.22 (IOVDD), U1.26 (RUN), U1.33 (IOVDD), U1.42 (IOVDD), U1.43 (ADC_AVDD), U1.44 (VREG_IN), U1.48 (USB_VDD), U1.49 (IOVDD)
- new net 3DS_C2: IC6.10 (VINC+), R20.1
- new net 3DS_C4: IC6.12 (VIND+), R21.2
- new net 3DS_SPX: IC6.2 (VINA+), R7.1
- new net 3DS_SPY: IC6.4 (VINB+), R8.1
- new net 3DS_TSXM: IC5.19 (A3)
- new net 3DS_TSXP: IC5.24 (B1)
- new net 3DS_TSYM: IC5.3 (A2)
- new net 3DS_TSYP: IC5.2 (B2)
- new net AGND: IC5.1 (AGND2), IC5.17 (AGND3), IC5.21 (AGND1), IC5.5 (AGND4), R13.1
- new net C2_RAW: C23.1, IC10.12 (OUT2(N.C.)), IC6.9 (VINC-), R22.1
- new net C4_RAW: C24.1, IC10.14 (OUT3_(N.C.)), IC6.13 (VIND-), R23.1
- new net I2C_SCL: IC10.2 (SCL)
- new net I2C_SDA: IC10.1 (SDA)
- new net LED_DIN: Q4.2 (S), R18.2
- new net LED_DIN_5V: LED1.1 (DIN), Q4.3 (D), R19.2
- new net QSPI_SCLK: IC1.6 (CLK), U1.52 (QSPI_SCLK)
- new net QSPI_SD0: IC1.5 (DI_(IO0)), U1.53 (QSPI_SD0)
- new net QSPI_SD1: IC1.2 (DO_(IO1)), U1.55 (QSPI_SD1)
- new net QSPI_SD2: IC1.3 (~{WP_(IO2)}), U1.54 (QSPI_SD2)
- new net QSPI_SD3: IC1.7 (~{HOLD_OR_RESET_(IO3)}), U1.51 (QSPI_SD3)
- new net QSPI_SS: IC1.1 (~{CS}), R2.2, U1.56 (QSPI_SS)
- new net SPI_CS: Q3.2 (S), R16.2
- new net SPI_CS_5V: IC5.11 (~{CS}), Q3.3 (D), R17.2
- new net SPI_SCK: Q1.2 (S), R9.2
- new net SPI_SCK_5V: IC5.14 (CLK), Q1.3 (D), R10.2
- new net SPI_TX: Q2.2 (S), R11.2
- new net SPI_TX_5V: IC5.12 (SDI), Q2.3 (D), R12.2
- new net SPST_IN: IC9.4 (IN)
- new net SPX_RAW: C18.2, IC10.8 (OUT0), IC6.1 (VINA-), R14.1
- new net SPY_RAW: C19.1, IC10.10 (OUT1), IC6.5 (VINB-), R15.1
- new net SWCLK: J5.3 (Pin_3), U1.24 (SWCLK)
- new net SWD: J5.1 (Pin_1), U1.25 (SWD)
- new net USB_DN_: J4.4 (Pin_4), R5.1
- new net USB_DP_: J4.3 (Pin_3), R4.1
- new net VOUTA: C18.1, IC3.1 (CCW), IC6.16 (VOUTA), R14.2
- new net VOUTB: C19.2, IC4.1 (CCW), IC6.6 (VOUTB), R15.2
- new net VOUTC: C23.2, IC6.8 (VOUTC), IC7.1 (CCW), R22.2
- new net VOUTD: C24.2, IC6.14 (VOUTD), IC8.1 (CCW), R23.2
- new net XIN: U1.20 (XIN), Y1.1 (INPUT)
- new net XOUT: R6.1, U1.21 (XOUT)
- no-connect marks 0 -> 12
Other:
- note added: "+"
- note added: "-"
- moved on the sheet: C14, C15, C16, C17, D1, D2, IC2, J2, U2

Commit message: WIP
Parts:
- removed C15: 10u, symbol Device:C_Small
- removed D1, D2: D_Shockley, symbol Device:D_Shockley
- added C3: 10u, Capacitor_SMD:C_0603_1608Metric, symbol Device:C_Small
- added D1, D2: D_Schottky, Diode_SMD:D_SOD-523, symbol Device:D_Schottky
- added J6: Conn_02x17_Counter_Clockwise, 5055503020:5055503020, symbol Connector_Generic:Conn_02x17_Counter_Clockwise
- added R13, R18: 510, Resistor_SMD:R_0201_0603Metric, symbol Device:R_Small
- C1: renamed from C14; footprint (none) -> Capacitor_SMD:C_0603_1608Metric; LCSC (none) -> C386081; Part (none) -> TMK107BBJ106MA-T
- C10: renamed from C19; footprint Capacitor_SMD:C_0603_1608Metric -> Capacitor_SMD:C_0201_0603Metric
- C11: renamed from C24; footprint Capacitor_SMD:C_0603_1608Metric -> Capacitor_SMD:C_0201_0603Metric
- C12: renamed from C13; footprint Capacitor_SMD:C_0402_1005Metric -> Capacitor_SMD:C_0201_0603Metric
- C13: renamed from C1; footprint Capacitor_SMD:C_0402_1005Metric -> Capacitor_SMD:C_0201_0603Metric
- C14: renamed from C2; footprint Capacitor_SMD:C_0402_1005Metric -> Capacitor_SMD:C_0201_0603Metric
- C15: renamed from C3; footprint Capacitor_SMD:C_0402_1005Metric -> Capacitor_SMD:C_0201_0603Metric
- C16: renamed from C4; footprint (none) -> Capacitor_SMD:C_0201_0603Metric
- C17: renamed from C5; value 1u -> 100n; footprint (none) -> Capacitor_SMD:C_0201_0603Metric
- C18: renamed from C22; footprint Capacitor_SMD:C_0402_1005Metric -> Capacitor_SMD:C_0201_0603Metric
- C19: renamed from C21; footprint Capacitor_SMD:C_0402_1005Metric -> Capacitor_SMD:C_0201_0603Metric
- C2: renamed from C20; footprint Capacitor_SMD:C_0603_1608Metric -> Capacitor_SMD:C_0201_0603Metric
- C20: renamed from C6; value 1u -> 100n; footprint (none) -> Capacitor_SMD:C_0201_0603Metric
- C21: renamed from C7; value 1u -> 100n; footprint (none) -> Capacitor_SMD:C_0201_0603Metric
- C22: renamed from C8; value 1u -> 100n; footprint (none) -> Capacitor_SMD:C_0201_0603Metric
- C23: renamed from C9; value 1u -> 100n; footprint (none) -> Capacitor_SMD:C_0201_0603Metric
- C24: renamed from C10; value 1u -> 100n; footprint (none) -> Capacitor_SMD:C_0201_0603Metric
- C25: renamed from C11; value 1u -> 100n; footprint (none) -> Capacitor_SMD:C_0201_0603Metric
- C4: renamed from C16; footprint (none) -> Capacitor_SMD:C_0201_0603Metric
- C5: renamed from C25; footprint Capacitor_SMD:C_0603_1608Metric -> Capacitor_SMD:C_0201_0603Metric
- C6: renamed from C18; footprint Capacitor_SMD:C_0603_1608Metric -> Capacitor_SMD:C_0201_0603Metric
- C7: renamed from C23; footprint Capacitor_SMD:C_0603_1608Metric -> Capacitor_SMD:C_0201_0603Metric
- C8: renamed from C17; footprint (none) -> Capacitor_SMD:C_0201_0603Metric
- C9: renamed from C12; footprint Capacitor_SMD:C_0402_1005Metric -> Capacitor_SMD:C_0201_0603Metric
- IC1: renamed from IC2; footprint XCL103D503CRG -> XCL103D503CR-G:XCL103D503CRG
- IC10: renamed from IC9; footprint SOT95P280X145-6N -> ADG801BRTZ-REEL7:SOT95P280X145-6N
- IC2: renamed from IC6; footprint QFN65P400X400X100-17N-D -> MCP659-E_ML:QFN65P400X400X100-17N-D
- IC4: renamed from IC1; footprint SON50P300X200X60-9N -> W25Q16JVUXIQ:SON50P300X200X60-9N
- IC5: renamed from IC3; footprint TC42X2102E -> TC42X-2-102E:TC42X2102E
- IC6: renamed from IC7; footprint TC42X2102E -> TC42X-2-102E:TC42X2102E
- IC7: renamed from IC4; footprint TC42X2102E -> TC42X-2-102E:TC42X2102E
- IC8: footprint TC42X2102E -> TC42X-2-102E:TC42X2102E
- IC9: renamed from IC5; footprint SOP65P640X120-24N -> AD8403ARUZ1-REEL:SOP65P640X120-24N
- J1: renamed from J2; footprint 2171790001_MOL -> 2171790001:2171790001_MOL
- J2: renamed from J3; footprint (none) -> Connector_PinHeader_1.27mm:PinHeader_1x04_P1.27mm_Vertical
- J3: renamed from J4; footprint (none) -> Connector_PinHeader_1.27mm:PinHeader_1x04_P1.27mm_Vertical
- J4: renamed from J1; footprint (none) -> Connector_PinHeader_1.27mm:PinHeader_1x02_P1.27mm_Vertical
- J5: footprint (none) -> Connector_PinHeader_1.27mm:PinHeader_1x03_P1.27mm_Vertical
- LED1: footprint SK6805EC15 -> SK6805-EC15:SK6805EC15
- R1, R15: footprint (none) -> Resistor_SMD:R_0201_0603Metric
- R10: renamed from R14; footprint (none) -> Resistor_SMD:R_0201_0603Metric
- R11: renamed from R20; footprint Resistor_SMD:R_0603_1608Metric -> Resistor_SMD:R_0201_0603Metric
- R12: renamed from R22; footprint (none) -> Resistor_SMD:R_0201_0603Metric
- R14: renamed from R8; footprint Resistor_SMD:R_0603_1608Metric -> Resistor_SMD:R_0201_0603Metric
- R16: renamed from R21; footprint Resistor_SMD:R_0603_1608Metric -> Resistor_SMD:R_0201_0603Metric
- R17: renamed from R23; footprint (none) -> Resistor_SMD:R_0201_0603Metric
- R19: renamed from R4; footprint Resistor_SMD:R_0402_1005Metric -> Resistor_SMD:R_0201_0603Metric
- R2: renamed from R3; footprint (none) -> Resistor_SMD:R_0201_0603Metric
- R20: renamed from R5; footprint Resistor_SMD:R_0402_1005Metric -> Resistor_SMD:R_0201_0603Metric
- R21: renamed from R13; footprint (none) -> Resistor_SMD:R_0201_0603Metric
- R22: renamed from R9; footprint (none) -> Resistor_SMD:R_0201_0603Metric
- R23: renamed from R16; footprint (none) -> Resistor_SMD:R_0201_0603Metric
- R24: renamed from R10; footprint (none) -> Resistor_SMD:R_0201_0603Metric
- R25: renamed from R17; footprint (none) -> Resistor_SMD:R_0201_0603Metric
- R26: renamed from R11; footprint (none) -> Resistor_SMD:R_0201_0603Metric
- R27: renamed from R18; footprint (none) -> Resistor_SMD:R_0201_0603Metric
- R28: renamed from R12; footprint (none) -> Resistor_SMD:R_0201_0603Metric
- R29: renamed from R19; footprint (none) -> Resistor_SMD:R_0201_0603Metric
- R3: renamed from R24; footprint Resistor_SMD:R_0603_1608Metric -> Resistor_SMD:R_0201_0603Metric
- R4: renamed from R25; footprint Resistor_SMD:R_0603_1608Metric -> Resistor_SMD:R_0201_0603Metric
- R5: renamed from R26; footprint Resistor_SMD:R_0603_1608Metric -> Resistor_SMD:R_0201_0603Metric
- R6: renamed from R27; footprint Resistor_SMD:R_0603_1608Metric -> Resistor_SMD:R_0201_0603Metric
- R7: renamed from R2; footprint Resistor_SMD:R_0402_1005Metric -> Resistor_SMD:R_0201_0603Metric
- R8: renamed from R6; footprint (none) -> Resistor_SMD:R_0201_0603Metric
- R9: renamed from R7; footprint Resistor_SMD:R_0603_1608Metric -> Resistor_SMD:R_0201_0603Metric
- U1: renamed from U2; footprint XDFN4_1X1_711AJ_ONS -> NCP167AMX330TBG:XDFN4_1X1_711AJ_ONS
- Y1: footprint AWSCR1200CELAC33T3 -> AWSCR-12.00CELA-C33-T3:AWSCR1200CELAC33T3
- renumbered IC10 to IC3, Q3 to Q2, Q2 to Q3, U1 to U2
Connections:
- net +5V: now also C3.1
- net 3DS_BTN0: now also U2.2 (GPIO0), J6.1 (Pin_1)
- net 3DS_BTN1: now also U2.3 (GPIO1), J6.2 (Pin_2)
- net 3DS_BTN10: now also U2.13 (GPIO10), J6.11 (Pin_11)
- net 3DS_BTN11: now also U2.14 (GPIO11), J6.12 (Pin_12)
- net 3DS_BTN12: now also U2.15 (GPIO12), J6.13 (Pin_13)
- net 3DS_BTN13: now also U2.16 (GPIO13), J6.14 (Pin_14)
- net 3DS_BTN14: now also U2.17 (GPIO14), J6.15 (Pin_15)
- net 3DS_BTN15: now also U2.18 (GPIO15), J6.16 (Pin_16)
- net 3DS_BTN2: now also U2.4 (GPIO2), J6.3 (Pin_3)
- net 3DS_BTN3: now also U2.5 (GPIO3), J6.4 (Pin_4)
- net 3DS_BTN4: now also U2.6 (GPIO4), J6.5 (Pin_5)
- net 3DS_BTN5: now also U2.7 (GPIO5), J6.6 (Pin_6)
- net 3DS_BTN6: now also U2.8 (GPIO6), J6.7 (Pin_7)
- net 3DS_BTN7: now also U2.9 (GPIO7), J6.8 (Pin_8)
- net 3DS_BTN8: now also U2.11 (GPIO8), J6.9 (Pin_9)
- net 3DS_BTN9: now also U2.12 (GPIO9), J6.10 (Pin_10)
- net 3DS_C2: now also J6.19 (Pin_19)
- net 3DS_C4: now also J6.20 (Pin_20)
- net 3DS_SPX: now also J6.17 (Pin_17)
- net 3DS_SPY: now also J6.18 (Pin_18)
- net 3DS_TSXM: now also J6.22 (Pin_22)
- net 3DS_TSXP: now also J6.21 (Pin_21)
- net 3DS_TSYM: now also J6.24 (Pin_24)
- net 3DS_TSYP: now also J6.23 (Pin_23)
- net 3DS_VBUS: now also D2.2 (A), J6.25 (Pin_25), J6.26 (Pin_26), J6.27 (Pin_27)
- net GND: now also C3.2, J6.28 (Pin_28), J6.29 (Pin_29), J6.30 (Pin_30), J6.31 (Pin_31), J6.32 (Pin_32), J6.33 (Pin_33), J6.34 (Pin_34)
- net I2C_SCL: now also U2.28 (GPIO17)
- net I2C_SDA: now also U2.27 (GPIO16)
- net LED_DIN: now also U2.34 (GPIO22)
- net LED_DIN_5V: now also R13.1; no longer LED1.1 (DIN)
- net SPI_CS: now also U2.31 (GPIO20)
- net SPI_SCK: now also U2.29 (GPIO18)
- net SPI_TX: now also U2.30 (GPIO19)
- net SPST_IN: now also U2.32 (GPIO21)
- net USB_VBUS_: now also D1.2 (A)
- net VIN: now also D1.1 (K), D2.1 (K)
- net at LED1.3 (DOUT): now also R18.1
- new net: LED1.1 (DIN), R13.2
- no-connect marks 12 -> 19
Other:
- moved on the sheet: C12

Commit message: WIP
Parts:
- J1: footprint 2171790001:2171790001_MOL -> my_2171790001:2171790001
- J2, J3: footprint Connector_PinHeader_1.27mm:PinHeader_1x04_P1.27mm_Vertical -> conn:PinHeader_1x04_P1.27mm_Vertical
- J4: footprint Connector_PinHeader_1.27mm:PinHeader_1x02_P1.27mm_Vertical -> conn:PinHeader_1x02_P1.27mm_Vertical
- J5: footprint Connector_PinHeader_1.27mm:PinHeader_1x03_P1.27mm_Vertical -> conn:PinHeader_1x03_P1.27mm_Vertical
Changed lines of the file:
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@@
 			)
 		)
-		(property "Footprint" "2171790001:2171790001_MOL"
+		(property "Footprint" "my_2171790001:2171790001"
 			(at 26.67 24.13 0)
 			(effects
@@
 			)
 		)
-		(property "Footprint" "Connector_PinHeader_1.27mm:PinHeader_1x04_P1.27mm_Vertical"
+		(property "Footprint" "conn:PinHeader_1x04_P1.27mm_Vertical"
 			(at 34.29 67.31 0)
 			(effects
@@
 			)
 		)
-		(property "Footprint" "Connector_PinHeader_1.27mm:PinHeader_1x04_P1.27mm_Vertical"
+		(property "Footprint" "conn:PinHeader_1x04_P1.27mm_Vertical"
 			(at 49.53 67.31 0)
 			(effects
@@
 			)
 		)
-		(property "Footprint" "Connector_PinHeader_1.27mm:PinHeader_1x03_P1.27mm_Vertical"
+		(property "Footprint" "conn:PinHeader_1x03_P1.27mm_Vertical"
 			(at 168.91 82.55 0)
 			(effects
@@
 			)
 		)
-		(property "Footprint" "Connector_PinHeader_1.27mm:PinHeader_1x02_P1.27mm_Vertical"
+		(property "Footprint" "conn:PinHeader_1x02_P1.27mm_Vertical"
 			(at 99.06 22.86 0)
 			(effects

Commit message: WIP
Connections:
- net GND: now also J3.3 (Pin_3); no longer J3.2 (Pin_2)
- net SPX_RAW: now also C6.1; no longer C6.2
- net USB_DN_: now also J3.2 (Pin_2); no longer J3.4 (Pin_4)
- net USB_DP_: now also J3.1 (Pin_1); no longer J3.3 (Pin_3)
- net USB_VBUS_: now also J3.4 (Pin_4); no longer J3.1 (Pin_1)
- net VOUTA: now also C6.2; no longer C6.1
Other:
- moved on the sheet: C6
Changed lines of the file:
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@@
 	(wire
 		(pts
-			(xy 64.77 72.39) (xy 64.77 67.31)
-		)
-		(stroke
-			(width 0)
-			(type default)
-		)
-	)
-	(wire
-		(pts
 			(xy 95.25 138.43) (xy 95.25 137.16)
 		)
@@
 	(wire
 		(pts
-			(xy 64.77 67.31) (xy 54.61 67.31)
-		)
-		(stroke
-			(width 0)
-			(type default)
-		)
-	)
-	(wire
-		(pts
 			(xy 31.75 132.08) (xy 45.72 132.08)
 		)
@@
 	(wire
 		(pts
+			(xy 54.61 69.85) (xy 64.77 69.85)
+		)
+		(stroke
+			(width 0)
+			(type default)
+		)
+	)
+	(wire
+		(pts
 			(xy 101.6 250.19) (xy 90.17 250.19)
 		)
@@
 	(wire
 		(pts
+			(xy 64.77 69.85) (xy 64.77 73.66)
+		)
+		(stroke
+			(width 0)
+			(type default)
+		)
+	)
+	(wire
+		(pts
 			(xy 209.55 193.04) (xy 181.61 193.04)
 		)
@@
 		)
 	)
+	(label "USB_VBUS_"
+		(at 54.61 72.39 0)
+		(fields_autoplaced yes)
+		(effects
+			(font
+				(size 1.27 1.27)
+			)
+			(justify left bottom)
+		)
+	)
 	(label "QSPI_SD0"
 		(at 248.92 81.28 180)
@@
 		)
 	)
-	(label "USB_VBUS_"
-		(at 54.61 64.77 0)
-		(fields_autoplaced yes)
-		(effects
-			(font
-				(size 1.27 1.27)
-			)
-			(justify left bottom)
-		)
-	)
 	(label "SPI_CS_5V"
 		(at 351.79 218.44 0)
@@
 		)
 	)
-	(label "USB_DN_"
-		(at 54.61 72.39 0)
-		(fields_autoplaced yes)
-		(effects
-			(font
-				(size 1.27 1.27)
-			)
-			(justify left bottom)
-		)
-	)
 	(label "3DS_BTN14"
 		(at 299.72 93.98 0)
@@
 		)
 	)
+	(label "USB_DP_"
+		(at 54.61 64.77 0)
+		(fields_autoplaced yes)
+		(effects
+			(font
+				(size 1.27 1.27)
+			)
+			(justify left bottom)
+		)
+	)
 	(label "SPY_RAW"
 		(at 173.99 194.31 270)
@@
 		)
 	)
-	(label "USB_DP_"
-		(at 54.61 69.85 0)
-		(fields_autoplaced yes)
-		(effects
-			(font
-				(size 1.27 1.27)
-			)
-			(justify left bottom)
-		)
-	)
 	(label "VINC+"
 		(at 68.58 187.96 0)
@@
 		)
 	)
+	(label "USB_DN_"
+		(at 54.61 67.31 0)
+		(fields_autoplaced yes)
+		(effects
+			(font
+				(size 1.27 1.27)
+			)
+			(justify left bottom)
+		)
+	)
 	(label "3DS_SPY"
 		(at 365.76 115.57 0)
@@
 	(symbol
 		(lib_id "Device:C_Small")
-		(at 125.73 184.15 270)
+		(at 125.73 184.15 90)
 		(mirror x)
 		(unit 1)
@@
 		(fields_autoplaced yes)
 		(property "Reference" "C6"
-			(at 125.7236 179.07 90)
+			(at 125.7363 177.8 90)
 			(effects
 				(font
@@
 		)
 		(property "Value" "10n"
-			(at 125.7236 181.61 90)
+			(at 125.7363 180.34 90)
 			(effects
 				(font
@@
 	(symbol
 		(lib_id "power:GND")
-		(at 64.77 72.39 0)
+		(at 64.77 73.66 0)
 		(unit 1)
 		(exclude_from_sim no)
@@
 		(fields_autoplaced yes)
 		(property "Reference" "#PWR04"
-			(at 64.77 78.74 0)
+			(at 64.77 80.01 0)
 			(effects
 				(font
@@
 		)
 		(property "Value" "GND"
-			(at 64.77 77.47 0)
+			(at 64.77 78.74 0)
 			(effects
 				(font
@@
 		)
 		(property "Footprint" ""
-			(at 64.77 72.39 0)
+			(at 64.77 73.66 0)
 			(effects
 				(font
@@
 		)
 		(property "Datasheet" ""
-			(at 64.77 72.39 0)
+			(at 64.77 73.66 0)
 			(effects
 				(font
@@
 		)
 		(property "Description" "Power symbol creates a global label with name \"GND\" , ground"
-			(at 64.77 72.39 0)
+			(at 64.77 73.66 0)
 			(effects
 				(font

Commit message: WIP
Connections:
- net 3DS_C4: now also R16.1; no longer R16.2
- net at IC8.2 (WIPER): now also R16.2; no longer R16.1
Other:
- moved on the sheet: R16
Changed lines of the file:
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@@
 	(symbol
 		(lib_id "Device:R_Small")
-		(at 179.07 218.44 270)
+		(at 179.07 218.44 90)
 		(unit 1)
 		(exclude_from_sim no)

Commit message: WIP
Connections:
- net +3.3V is gone; now on net +3V3: C4.1, Q1.1 (G), Q2.1 (G), Q3.1 (G), Q4.1 (G), R22.1, R23.1, R26.1, R27.1, U1.1 (OUT)
- net 3DS_BTN0: now also J6.30 (Pin_30); no longer J6.1 (Pin_1)
- net 3DS_BTN1: now also J6.29 (Pin_29); no longer J6.2 (Pin_2)
- net 3DS_BTN10: now also J6.20 (Pin_20); no longer J6.11 (Pin_11)
- net 3DS_BTN11: now also J6.19 (Pin_19); no longer J6.12 (Pin_12)
- net 3DS_BTN12: now also J6.17 (Pin_17); no longer J6.13 (Pin_13)
- net 3DS_BTN13: now also J6.18 (Pin_18); no longer J6.14 (Pin_14)
- net 3DS_BTN14: now also J6.16 (Pin_16); no longer J6.15 (Pin_15)
- net 3DS_BTN15: now also J6.7 (Pin_7); no longer J6.16 (Pin_16)
- net 3DS_BTN2: now also J6.28 (Pin_28); no longer J6.3 (Pin_3)
- net 3DS_BTN3: now also J6.27 (Pin_27); no longer J6.4 (Pin_4)
- net 3DS_BTN4: now also J6.26 (Pin_26); no longer J6.5 (Pin_5)
- net 3DS_BTN5: now also J6.25 (Pin_25); no longer J6.6 (Pin_6)
- net 3DS_BTN6: now also J6.24 (Pin_24); no longer J6.7 (Pin_7)
- net 3DS_BTN7: now also J6.23 (Pin_23); no longer J6.8 (Pin_8)
- net 3DS_BTN8: now also J6.22 (Pin_22); no longer J6.9 (Pin_9)
- net 3DS_BTN9: now also J6.21 (Pin_21); no longer J6.10 (Pin_10)
- net 3DS_C2: now also J6.13 (Pin_13); no longer J6.19 (Pin_19)
- net 3DS_C4: now also J6.12 (Pin_12); no longer J6.20 (Pin_20)
- net 3DS_SPX: now also J6.15 (Pin_15); no longer J6.17 (Pin_17)
- net 3DS_SPY: now also J6.14 (Pin_14); no longer J6.18 (Pin_18)
- net 3DS_TSXM: now also J6.10 (Pin_10); no longer J6.22 (Pin_22)
- net 3DS_TSXP: now also J6.11 (Pin_11); no longer J6.21 (Pin_21)
- net 3DS_TSYM: now also J6.8 (Pin_8); no longer J6.24 (Pin_24)
- net 3DS_TSYP: now also J6.9 (Pin_9); no longer J6.23 (Pin_23)
- net 3DS_VBUS: now also J6.4 (Pin_4), J6.5 (Pin_5), J6.6 (Pin_6); no longer J6.25 (Pin_25), J6.26 (Pin_26), J6.27 (Pin_27)
- net GND: now also J6.1 (Pin_1), J6.2 (Pin_2), J6.3 (Pin_3); no longer J6.28 (Pin_28), J6.29 (Pin_29), J6.30 (Pin_30)
- net I2C_SCL: now also U2.27 (GPIO16); no longer U2.28 (GPIO17)
- net I2C_SDA: now also U2.28 (GPIO17); no longer U2.27 (GPIO16)
- net LED_DIN: now also U2.29 (GPIO18); no longer U2.34 (GPIO22)
- net SPI_CS: now also U2.34 (GPIO22); no longer U2.31 (GPIO20)
- net SPI_SCK: now also U2.31 (GPIO20); no longer U2.29 (GPIO18)
- net SPI_TX: now also U2.32 (GPIO21); no longer U2.30 (GPIO19)
- net SPST_IN: now also U2.30 (GPIO19); no longer U2.32 (GPIO21)
- net USB_DN: now also J2.2 (Pin_2); no longer J2.4 (Pin_4)
- net USB_DP: now also J2.1 (Pin_1); no longer J2.3 (Pin_3)
- net USB_GND: now also J2.3 (Pin_3); no longer J2.2 (Pin_2)
- net USB_VBUS: now also J2.4 (Pin_4); no longer J2.1 (Pin_1)

Commit message: WIP
Connections:
- net 3DS_TSXM: now also J6.9 (Pin_9); no longer J6.10 (Pin_10)
- net 3DS_TSXP: now also J6.8 (Pin_8); no longer J6.11 (Pin_11)
- net 3DS_TSYM: now also J6.11 (Pin_11); no longer J6.8 (Pin_8)
- net 3DS_TSYP: now also J6.10 (Pin_10); no longer J6.9 (Pin_9)
Changed lines of the file:
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@@
+		)
+	)
+	(label "3DS_TSXP"
+		(at 353.06 92.71 180)
+		(fields_autoplaced yes)
+		(effects
+			(font
+				(size 1.27 1.27)
+			)
+			(justify right bottom)
 		)
 	)
@@
 		)
 	)
+	(label "3DS_TSYP"
+		(at 353.06 97.79 180)
+		(fields_autoplaced yes)
+		(effects
+			(font
+				(size 1.27 1.27)
+			)
+			(justify right bottom)
+		)
+	)
 	(label "3DS_BTN1"
 		(at 299.72 60.96 0)
@@
 		)
 	)
-	(label "3DS_TSXP"
-		(at 353.06 100.33 180)
-		(fields_autoplaced yes)
-		(effects
-			(font
-				(size 1.27 1.27)
-			)
-			(justify right bottom)
-		)
-	)
 	(label "QSPI_SD0"
 		(at 248.92 81.28 180)
@@
 		)
 	)
+	(label "3DS_TSXM"
+		(at 353.06 95.25 180)
+		(fields_autoplaced yes)
+		(effects
+			(font
+				(size 1.27 1.27)
+			)
+			(justify right bottom)
+		)
+	)
 	(label "3DS_BTN2"
 		(at 299.72 63.5 0)
@@
 		)
 	)
-	(label "3DS_TSYP"
-		(at 353.06 95.25 180)
-		(fields_autoplaced yes)
-		(effects
-			(font
-				(size 1.27 1.27)
-			)
-			(justify right bottom)
-		)
-	)
 	(label "3DS_BTN11"
 		(at 299.72 86.36 0)
@@
 		)
 	)
-	(label "3DS_TSYM"
-		(at 353.06 92.71 180)
-		(fields_autoplaced yes)
-		(effects
-			(font
-				(size 1.27 1.27)
-			)
-			(justify right bottom)
-		)
-	)
 	(label "AGND"
 		(at 283.21 185.42 0)
@@
 		)
 	)
-	(label "3DS_TSXM"
-		(at 353.06 97.79 180)
-		(fields_autoplaced yes)
-		(effects
-			(font
-				(size 1.27 1.27)
-			)
-			(justify right bottom)
-		)
-	)
 	(label "3DS_TSYP"
 		(at 252.73 180.34 180)
@@
 		)
 	)
+	(label "3DS_TSYM"
+		(at 353.06 100.33 180)
+		(fields_autoplaced yes)
+		(effects
+			(font
+				(size 1.27 1.27)
+			)
+			(justify right bottom)
+		)
+	)
